File: hardware/control-io/control-io.kicad_sch (KiCad schematic)
At the start: 30 parts, among them J1 3.5mm TRS MIDI IN, J2 6.35mm TRS EXPRESSION, J3 RASPBERRY PI CONTROL HEADER, SW1A DPDT POLARITY — POLE A, SW1B DPDT POLARITY — POLE B, U1 6N138, U2 ADS1115IDGS (ADDR=GND / 0x48)

Commit message: fix: code review fixes
Parts:
- removed GND (x4): GND, symbol Custom:rail_down
- removed SW1A: DPDT POLARITY — POLE A, symbol Device:U_DPDT_POLARITY_—_POLE_A
- removed SW1B: DPDT POLARITY — POLE B, symbol Device:U_DPDT_POLARITY_—_POLE_B
- removed U2: ADS1115IDGS (ADDR=GND / 0x48), symbol Device:U_ADS1115IDGS_(ADDR=GND_0x48)
- removed V3V3 (x4): V3V3, symbol Custom:rail_up
- removed V5 (x2): V5, symbol Custom:rail_up
- removed VEXP: VEXP, symbol Custom:rail_up
- added GND (x4): GND, symbol Custom:rail_down
- added SW1A: DPDT POLE A, symbol Device:U_DPDT_POLE_A
- added SW1B: DPDT POLE B, symbol Device:U_DPDT_POLE_B
- added U2: ADS1115 (0x48), symbol Device:U_ADS1115_(0x48)
- added V3V3 (x4): V3V3, symbol Custom:rail_up
- added V5 (x2): V5, symbol Custom:rail_up
- added VEXP (x2): VEXP, symbol Custom:rail_up
Connections:
- net ADC_ALERT: now also U2.2 (ALERT)
- net ADC_FILTER: now also U2.4 (AIN0)
- net ADC_SENSE: now also R5.1, SW1A.3 (POS_B), SW1B.2 (POS_A)
- net EXP_RING: now also SW1B.1 (COM)
- net EXP_TIP: now also SW1A.1 (COM)
- net I2C_SCL: now also U2.10 (SCL)
- net I2C_SDA: now also U2.9 (SDA)
- net at C1.1, U1.8 (VCC): now also V5.1
- net at C1.2, R2.2: now also U1.5 (GND), GND.1
- net at R4.2: now also VEXP.1
- net at J3.2 (3V3): now also V3V3.1
- net at J2.3 (SLEEVE), J3.3 (GND): now also GND.1
- net at J3.1 (5V): now also V5.1
- net at R6.1: now also C3.1, U2.8 (VDD), V3V3.1
- net at R4.1: now also V3V3.1
- net at R3.1: now also V3V3.1
- net at C3.2: now also GND.1, U2.3 (GND)
- new net: SW1A.2 (POS_A), SW1B.3 (POS_B), VEXP.1
- new net: GND.1, U2.1 (ADDR), U2.5 (AIN1), U2.6 (AIN2), U2.7 (AIN3)
Other:
- note added: "HOST: Raspberry Pi GPIO header"
- note added: "I2C pull-ups are already present on the host bus."
- note removed: "HOST: Raspberry Pi header — UART4 RX GPIO9; I2C1 GPIO2/GPIO3"
- note removed: "I2C pull-ups are already present on the host bus; do not fit duplicates unless measured."

Commit message: feat: add control I/O board and fail-safe audio relay control (#45)
- Add complete control-I/O hardware design, schematics, harnesses, and wiring documentation
- Add GPIO10 default-low relay control with kernel LED support and supervised mute handling
- Add connectivity checker and update build configuration for the new hardware
Parts:
- removed D2, D3: D, symbol Device:schottky_diode_right
- removed GND (x4): GND, symbol Custom:rail_down
- removed J1: 3.5mm TRS MIDI IN, symbol Device:U_3.5mm_TRS_MIDI_IN
- removed J2: 6.35mm TRS EXPRESSION, symbol Device:U_6.35mm_TRS_EXPRESSION
- removed J3: RASPBERRY PI CONTROL HEADER, symbol Device:U_RASPBERRY_PI_CONTROL_HEADER
- removed SW1A: DPDT POLE A, symbol Device:U_DPDT_POLE_A
- removed SW1B: DPDT POLE B, symbol Device:U_DPDT_POLE_B
- removed U1: 6N138, symbol Device:U_6N138
- removed U2: ADS1115 (0x48), symbol Device:U_ADS1115_(0x48)
- removed V3V3 (x4): V3V3, symbol Custom:rail_up
- removed V5 (x2): V5, symbol Custom:rail_up
- removed VEXP (x2): VEXP, symbol Custom:rail_up
- added AGND (x5): AGND, symbol Custom:rail_down
- added C10, C13, C15, C21, C24, C26, C28, C29: 100nF, symbol Device:capacitor_right
- added C11: 1nF 1kV, symbol Device:capacitor_right
- added C12, C14, C22, C25: 1uF, symbol Device:capacitor_right
- added C20: 22uF, symbol Device:capacitor_right
- added C23: 10uF, symbol Device:capacitor_right
- added C27: 4.7nF 1kV, symbol Device:capacitor_right
- added C4, C5, C6: 2.2uF FILM, symbol Device:capacitor_right
- added C7, C8, C9: 10uF BIPOLAR, symbol Device:capacitor_right
- added D10, D2: BAT54S, symbol Device:U_BAT54S
- added D11, D12, D13, D14, D15, D16, D17, D18, D3, D4, D5, D6, D7, D8, D9: D, symbol Device:diode_right
- added F1: F1, symbol Device:fuse_horz
- added F2: F2, symbol Device:fuse_horz
- added FB1: BLM21PG221SN1D, symbol Device:U_BLM21PG221SN1D
- added J1, J5: B2B-XH-A(LF)(SN) / PANEL TS HARNESS, symbol Device:U_B2B-XH-A(LF)(SN)_PANEL_TS_HARNESS
- added J2: 22-27-2041 / CODEC ZERO P1 HARNESS, symbol Device:U_22-27-2041_CODEC_ZERO_P1_HARNESS
- added J3: 22-27-2041 / CODEC ZERO P2 HARNESS, symbol Device:U_22-27-2041_CODEC_ZERO_P2_HARNESS
- added J4: B3B-XH-A(LF)(SN) / PANEL TRS HARNESS, symbol Device:U_B3B-XH-A(LF)(SN)_PANEL_TRS_HARNESS
- added J6: B3B-XH-A(LF)(SN) / PANEL MIDI HARNESS, symbol Device:U_B3B-XH-A(LF)(SN)_PANEL_MIDI_HARNESS
- added J7: B3B-XH-A(LF)(SN) / PANEL EXP HARNESS, symbol Device:U_B3B-XH-A(LF)(SN)_PANEL_EXP_HARNESS
- added J8: 2x20 STACK-THROUGH, symbol Device:U_2x20_STACK-THROUGH
- added J9: CHASSIS STUD, symbol Device:U_CHASSIS_STUD
- added K1, K2: ATQ209 / TQ2-5V, symbol Device:U_ATQ209_TQ2-5V
- added Q1: AO3400A, symbol Device:U_AO3400A
- added R10, R11: 20kΩ, symbol Device:boxresistor_right
- added R12, R32, R35: 10kΩ, symbol Device:boxresistor_right
- added R13, R14, R15: 100Ω, symbol Device:boxresistor_right
- added R16, R17, R18, R36, R37, R38, R7, R8, R9: 100kΩ, symbol Device:boxresistor_right
- added R19, R21, R33: 220Ω, symbol Device:boxresistor_right
- added R20, R24: 4.7kΩ, symbol Device:boxresistor_right
- added R22, R30: 1MΩ, symbol Device:boxresistor_right
- added R23, R27, R28, R29, R34: 1kΩ, symbol Device:boxresistor_right
- added R25, R26: 33Ω, symbol Device:boxresistor_right
- added R31: 0Ω, symbol Device:boxresistor_right
- added SW1: JS202011CQN, symbol Device:U_JS202011CQN
- added U1: OPA4377AIPWR, symbol Device:U_OPA4377AIPWR
- added U2: TPS7A2045PDBVR, symbol Device:U_TPS7A2045PDBVR
- added U3: TLE2426IDR, symbol Device:U_TLE2426IDR
- added U4: H11L1M, symbol Device:U_H11L1M
- added U5: ADS1115IDGSR (0x48), symbol Device:U_ADS1115IDGSR_(0x48)
- added V4V5_A: V4V5_A, symbol Custom:rail_up
- C1: value 100nF -> 220nF FILM
- C2: value 100nF -> 100pF C0G
- C3: value 100nF -> 2.2uF FILM
- R1: value 220Ω -> 1kΩ
- R2: value 10kΩ -> 1MΩ
- R3: value 4.7kΩ -> 10kΩ
- R4: value 1kΩ -> 100Ω
- R5: value 4.7kΩ -> 100kΩ
- R6: value 10kΩ -> 100Ω
Connections:
- net ADC_SENSE is gone; now on net CODEC_IN_L: R5.1
- net OPTO_BASE is gone; now on net GUITAR_BIAS: R2.1
- net EXP_RING: now also D9.2, J7.2 (RING), SW1.6 (COM_B)
- net EXP_TIP: now also D8.2, J7.1 (TIP), SW1.3 (COM_A)
- net MIDI_LED_A: now also D7.2, R19.2, U4.1 (LED_A); no longer D1.2, R1.2
- net V3V3: now also C10.1, C14.1, C15.1, D10.3 (HIGH), D17.1, J8.1 (3V3), J8.17 (3V3_2), R20.1, R32.1, U4.6 (VCC), U5.8 (VDD)
- net CODEC_IN_R_AC: now reaches R6.1
- net CODEC_IN_R_AC: now also C4.2; no longer C3.1
- net CODEC_IN_L_AC: now reaches C3.2
- net CODEC_IN_L_AC: now also R4.1
- net GUITAR_BIAS: now reaches C1.2
- net GUITAR_BIAS: now also R3.1; no longer R2.2
- net at C1.1: now also R1.2
- net CODEC_IN_L: now reaches R4.2
- net CODEC_IN_L: now also J2.1 (LEFT)
- net VREF_2V25: now reaches C2.2
- net VREF_2V25: now also R2.2, R8.2, R9.2, U1.12 (IN_PLUS_D), U3.1 (OUT)
- net ADC_ALERT renamed CODEC_IN_R
- net CODEC_IN_R: now also J2.3 (RIGHT), R7.1
- net ADC_FILTER: no longer names the net of R5.2
- net ADC_FILTER: now also J2.2 (GND_L), J2.4 (GND_R), R7.2; no longer C2.1
- net MIDI_RX renamed GUITAR_PROTECTED
- net GUITAR_PROTECTED: now also C2.1, D2.2 (IO), U1.3 (IN_PLUS_A)
- net MIDI_SINK_TIP renamed CHASSIS
- net CHASSIS: now also C11.2, C27.1, D18.1, D3.1, D4.1, D5.1, D8.1, D9.1, J9.1 (CHASSIS), R22.2, R30.1, R31.1
- net MIDI_SOURCE_RING renamed GUITAR_TIP
- net GUITAR_TIP: now also D1.2, J1.1 (TIP)
- new net: C8.2, R14.1
- new net: AGND.1, C13.2, D18.2
- new net: R32.2, R33.1, U5.2 (ALERT)
- new net: U2.1 (IN), U2.3 (EN)
- new net: C21.2, U2.2 (GND)
- new net: AGND.1, C14.2, C15.2, R27.2, R28.2, R29.2, U5.3 (GND)
- new net: AGND.1, C20.2, D2.1 (LOW)
- new net: C28.1, D2.3 (HIGH)
- new net: F1.1, F2.1, J8.2 (5V), J8.4 (5V_2)
- new net: C7.2, R13.1
- new net: J1.2 (SLEEVE), J8.25 (GND_5), J8.39 (GND_8), J8.9 (GND_2)
- new net: AGND.1, C27.2, R30.2, R31.2
- new net: K1.3 (COM_A), R36.1
- new net: K1.8 (COM_B), R14.2
- new net: C9.2, R15.1
- new net: D10.2 (IO), R24.2
- new net ADC_ALERT_GPIO: J8.22 (GPIO25_ADC_ALERT), R33.2
- new net ADC_UNUSED_1: R27.1, U5.5 (AIN1)
- new net ADC_UNUSED_2: R28.1, U5.6 (AIN2)
- new net ADC_UNUSED_3: R29.1, U5.7 (AIN3)
- new net AGND: C10.2, C12.2, C22.2, C23.2, C24.2, C25.2, C26.2, C28.2, C29.2, D10.1 (LOW), J3.2 (GND_L), J3.4 (GND_R), J4.3 (SLEEVE), J5.2 (SLEEVE), J7.3 (SLEEVE), J8.14 (GND_3), J8.20 (GND_4), J8.30 (GND_6), J8.34 (GND_7), J8.6 (GND), Q1.2 (S), R16.2, R17.2, R18.2, R35.2, R36.2, R37.2, R38.2, U1.11 (VMINUS), U3.2 (COMMON), U4.4 (GND), U5.1 (ADDR)
- new net AMP_OUT: D5.2, J5.1 (TIP), K2.7 (NO_B), R18.1
- new net AMP_RELAY_IN: K2.3 (COM_A), K2.8 (COM_B), R38.1
- new net CODEC_OUT_L: C5.1, J3.1 (LEFT)
- new net CODEC_OUT_L_BIAS: C5.2, R8.1, U1.5 (IN_PLUS_B)
- new net CODEC_OUT_R: C6.1, J3.3 (RIGHT)
- new net CODEC_OUT_R_BIAS: C6.2, R9.1, U1.10 (IN_PLUS_C)
- new net EXP_ADC_FILTER: C13.1, U5.4 (AIN0)
- new net EXP_SENSE: R24.1, SW1.2 (B_A), SW1.4 (A_B)
- new net GPIO10_MUTE: J8.19 (GPIO10_MUTE), R34.1
- new net GUITAR_BUFFERED: C3.1, C4.1, U1.1 (OUT_A), U1.2 (IN_MINUS_A)
- new net I2C_SCL_ADC: R26.2, U5.10 (SCL)
- new net I2C_SCL_HOST: J8.5 (GPIO3_SCL), R26.1
- new net I2C_SDA_ADC: R25.2, U5.9 (SDA)
- new net I2C_SDA_HOST: J8.3 (GPIO2_SDA), R25.1
- new net LINE_L_BUFFERED: C7.1, R10.1, U1.6 (IN_MINUS_B), U1.7 (OUT_B)
- new net LINE_L_RELAY_IN: R13.2
- new net LINE_OUT_L: D3.2, J4.1 (TIP_L), R16.1
- new net LINE_OUT_R: D4.2, J4.2 (RING_R), R17.1
- new net LINE_R_BUFFERED: C8.1, R11.1, U1.9 (IN_MINUS_C)
- new net LINE_R_RELAY_IN: R37.1
- new net MIDI_BRIDGE_NEG: D15.1, D16.1, D7.1, U4.2 (LED_K)
- new net MIDI_BRIDGE_POS: D13.2, D14.2, R19.1
- new net MIDI_RING_ISO: D14.1, D16.2, D6.2, J6.2 (RING)
- new net MIDI_RX_GPIO: J8.21 (GPIO9_UART4_RX), R21.2
- new net MIDI_RX_RAW: R20.2, R21.1, U4.5 (VO)
- new net MIDI_SHIELD: C11.1, J6.3 (SLEEVE), R22.1
- new net MIDI_TIP_ISO: D13.1, D15.2, D6.1, J6.1 (TIP)
- new net MONO_BUFFERED: C9.1, R12.2, U1.14 (OUT_D)
- new net MONO_SUM_NODE: R10.2, R11.2, R12.1, U1.13 (IN_MINUS_D)
- new net RELAY_CLAMP_MID: D11.2, D12.2
- new net RELAY_COIL_LOW: D11.1, K1.10 (COIL_N), K2.10 (COIL_N), Q1.3 (D)
- new net RELAY_GATE: Q1.1 (G), R34.2, R35.1
- new net V4V5_A: C23.1, C24.1, C26.1, C29.1, U1.4 (VPLUS), U2.5 (OUT), U3.3 (IN)
- new net V5_FILTERED: C20.1, C21.1, C22.1, FB1.2 (OUT)
- new net V5_FUSED: F1.2, FB1.1 (IN)
- new net V5_RELAY_FUSED: D12.1, F2.2, K1.1 (COIL_P), K2.1 (COIL_P)
- new net VEXP: C12.1, R23.2, SW1.1 (A_A), SW1.5 (B_B)
- new net VEXP_SOURCE: D17.2, R23.1
- new net VREF_NR: C25.1, U3.5 (NOISE_REDUCTION)
Other:
- note added: "1. POWER / REFERENCE / CHASSIS"
- note added: "2. HIGH-Z GUITAR INPUT → CODEC ZERO AUX IN"
- note added: "3. CODEC ZERO AUX OUT → STEREO LINE + MONO GUITAR AMP"
- note added: "4. GALVANICALLY ISOLATED TRS MIDI INPUT"
- note added: "5. PROTECTED PASSIVE EXPRESSION PEDAL INPUT"
- note added: "6. FAIL-SAFE OUTPUT MUTE"
- note added: "ARDOR PROFESSIONAL AUDIO + CONTROL I/O FOR RASPBERRY PI / CODEC ZERO"
- note added: "Codec P1/P2 pin order (square pin 1): LEFT, GND, RIGHT, GND. AUX maximum: 1 V RMS."
- note added: "GPIO10 HIGH closes K1/K2 only after codec clocks and bias are stable; GPIO10 defaults LOW at reset."
- note added: "MIDI cable side is isolated: never join MIDI_TIP/RING/SHIELD to AGND/DGND. No extra I2C pull-ups fitted."
- note added: "Rev B — fail-safe mute, bipolar audio ESD, protected guitar/line/amp, isolated MIDI, expression ADC"
- note added: "U1 is one OPA4377AIPWR in TSSOP-14; place 100nF directly at pins 4 and 11."
- note added: "Use isolated-bushing audio jacks. Bond CHASSIS at J9; fit R31 only after hum/EMC verification."
- note removed: "ARDOR CONTROL I/O — TRS-A MIDI IN + EXPRESSION ADC"
- note removed: "EXPRESSION: passive 6.35 mm TRS pedal, hardware polarity selector, ADS1115"
- note removed: "HOST: Raspberry Pi GPIO header"
- note removed: "I2C pull-ups are already present on the host bus."
- note removed: "MIDI IN: 3.5 mm TRS Type A, galvanically isolated"
- note removed: "R4 limits a shorted pedal cable to 3.3 mA. D2/D3: BAT54 Schottky clamps."
- note removed: "SW1A/SW1B are the two mechanically linked poles of one DPDT switch."

Commit message: Feature/control io revc (#46)
* feat(hardware): add Rev C integrated codec design

- Add generated Rev C DA7212 schematic and KiCad project files
- Add codec connectivity checks, wiring map, and fabrication release guidance
- Support reusable schematic generation and Rev C package scripts

* feat: add reviewed Rev B control I/O schematic package

- Split the design into eight hierarchical functional sheets
- Correct component pinouts, footprints, connectivity, and documentation
- Add automated review gates and Rev B electrical audit
Parts:
- removed AGND (x5): AGND, symbol Custom:rail_down
- removed C1: 220nF FILM, symbol Device:capacitor_right
- removed C10, C13, C15, C21, C24, C26, C28, C29: 100nF, symbol Device:capacitor_right
- removed C11: 1nF 1kV, symbol Device:capacitor_right
- removed C12, C14, C22, C25: 1uF, symbol Device:capacitor_right
- removed C2: 100pF C0G, symbol Device:capacitor_right
- removed C20: 22uF, symbol Device:capacitor_right
- removed C23: 10uF, symbol Device:capacitor_right
- removed C27: 4.7nF 1kV, symbol Device:capacitor_right
- removed C3, C4, C5, C6: 2.2uF FILM, symbol Device:capacitor_right
- removed C7, C8, C9: 10uF BIPOLAR, symbol Device:capacitor_right
- removed D1, D11, D12, D13, D14, D15, D16, D17, D18, D3, D4, D5, D6, D7, D8, D9: D, symbol Device:diode_right
- removed D10, D2: BAT54S, symbol Device:U_BAT54S
- removed F1: F1, symbol Device:fuse_horz
- removed F2: F2, symbol Device:fuse_horz
- removed FB1: BLM21PG221SN1D, symbol Device:U_BLM21PG221SN1D
- removed J1, J5: B2B-XH-A(LF)(SN) / PANEL TS HARNESS, symbol Device:U_B2B-XH-A(LF)(SN)_PANEL_TS_HARNESS
- removed J2: 22-27-2041 / CODEC ZERO P1 HARNESS, symbol Device:U_22-27-2041_CODEC_ZERO_P1_HARNESS
- removed J3: 22-27-2041 / CODEC ZERO P2 HARNESS, symbol Device:U_22-27-2041_CODEC_ZERO_P2_HARNESS
- removed J4: B3B-XH-A(LF)(SN) / PANEL TRS HARNESS, symbol Device:U_B3B-XH-A(LF)(SN)_PANEL_TRS_HARNESS
- removed J6: B3B-XH-A(LF)(SN) / PANEL MIDI HARNESS, symbol Device:U_B3B-XH-A(LF)(SN)_PANEL_MIDI_HARNESS
- removed J7: B3B-XH-A(LF)(SN) / PANEL EXP HARNESS, symbol Device:U_B3B-XH-A(LF)(SN)_PANEL_EXP_HARNESS
- removed J8: 2x20 STACK-THROUGH, symbol Device:U_2x20_STACK-THROUGH
- removed J9: CHASSIS STUD, symbol Device:U_CHASSIS_STUD
- removed K1, K2: ATQ209 / TQ2-5V, symbol Device:U_ATQ209_TQ2-5V
- removed Q1: AO3400A, symbol Device:U_AO3400A
- removed R1, R23, R27, R28, R29, R34: 1kΩ, symbol Device:boxresistor_right
- removed R10, R11: 20kΩ, symbol Device:boxresistor_right
- removed R12, R3, R32, R35: 10kΩ, symbol Device:boxresistor_right
- removed R13, R14, R15, R4, R6: 100Ω, symbol Device:boxresistor_right
- removed R16, R17, R18, R36, R37, R38, R5, R7, R8, R9: 100kΩ, symbol Device:boxresistor_right
- removed R19, R21, R33: 220Ω, symbol Device:boxresistor_right
- removed R2, R22, R30: 1MΩ, symbol Device:boxresistor_right
- removed R20, R24: 4.7kΩ, symbol Device:boxresistor_right
- removed R25, R26: 33Ω, symbol Device:boxresistor_right
- removed R31: 0Ω, symbol Device:boxresistor_right
- removed SW1: JS202011CQN, symbol Device:U_JS202011CQN
- removed U1: OPA4377AIPWR, symbol Device:U_OPA4377AIPWR
- removed U2: TPS7A2045PDBVR, symbol Device:U_TPS7A2045PDBVR
- removed U3: TLE2426IDR, symbol Device:U_TLE2426IDR
- removed U4: H11L1M, symbol Device:U_H11L1M
- removed U5: ADS1115IDGSR (0x48), symbol Device:U_ADS1115IDGSR_(0x48)
- removed V4V5_A: V4V5_A, symbol Custom:rail_up
Other:
- added sheet codec_output_processing (codec_output_processing.kicad_sch)
- added sheet expression_input (expression_input.kicad_sch)
- added sheet gpio_header (gpio_header.kicad_sch)
- added sheet guitar_input (guitar_input.kicad_sch)
- added sheet midi_input (midi_input.kicad_sch)
- added sheet output_mute (output_mute.kicad_sch)
- added sheet power_reference (power_reference.kicad_sch)
- added sheet relay_outputs (relay_outputs.kicad_sch)
- note removed: "1. POWER / REFERENCE / CHASSIS"
- note removed: "2. HIGH-Z GUITAR INPUT → CODEC ZERO AUX IN"
- note removed: "3. CODEC ZERO AUX OUT → STEREO LINE + MONO GUITAR AMP"
- note removed: "4. GALVANICALLY ISOLATED TRS MIDI INPUT"
- note removed: "5. PROTECTED PASSIVE EXPRESSION PEDAL INPUT"
- note removed: "6. FAIL-SAFE OUTPUT MUTE"
- note removed: "ARDOR PROFESSIONAL AUDIO + CONTROL I/O FOR RASPBERRY PI / CODEC ZERO"
- note removed: "Codec P1/P2 pin order (square pin 1): LEFT, GND, RIGHT, GND. AUX maximum: 1 V RMS."
- note removed: "GPIO10 HIGH closes K1/K2 only after codec clocks and bias are stable; GPIO10 defaults LOW at reset."
- note removed: "MIDI cable side is isolated: never join MIDI_TIP/RING/SHIELD to AGND/DGND. No extra I2C pull-ups fitted."
- note removed: "Rev B — fail-safe mute, bipolar audio ESD, protected guitar/line/amp, isolated MIDI, expression ADC"
- note removed: "U1 is one OPA4377AIPWR in TSSOP-14; place 100nF directly at pins 4 and 11."
- note removed: "Use isolated-bushing audio jacks. Bond CHASSIS at J9; fit R31 only after hum/EMC verification."
