File: hardware/aaa/ardor-io/02_MIDI.kicad_sch (KiCad schematic)
At the start: 16 parts, among them J201 MIDI IN - PANEL DIN, J202 TO MIDI PANEL / 4,5, U201 H11L1M

Commit message: feat: finalize Ardor IO hardware rev2 production package
- Update schematics, PCB, BOM, and documentation
- Add assembly exports, review artifacts, and verification data
Parts:
- C201: value 100n / 16V -> 100n / 50V X7R; JLCPCB Part # (none) -> C14663; MPN (none) -> YAGEO CC0603KRX7R9BB104
- C202, C203: JLCPCB Part # (none) -> C367316; MPN (none) -> CCTC TCC1206COG101J102DT
- D201: JLCPCB Part # (none) -> C81598; MPN 1N4148W -> ST(Semtech) 1N4148W
- D202: JLCPCB Part # (none) -> C19224; MPN Nexperia PESD5V0S1BA -> Nexperia PESD5V0S1BA,115
- D203, D204: JLCPCB Part # (none) -> C69324; MPN Nexperia PESD24VL1BA -> Nexperia PESD24VL1BA,115
- FB201, FB202: JLCPCB Part # (none) -> C19330
- R201: JLCPCB Part # (none) -> C22962; MPN (none) -> UNI-ROYAL 0603WAF2200T5E
- R202: JLCPCB Part # (none) -> C21190; MPN (none) -> UNI-ROYAL 0603WAF1001T5E
- R203: JLCPCB Part # (none) -> C22775; MPN (none) -> UNI-ROYAL 0603WAF1000T5E
Other:
- note added: "Female DIN, 180 degrees. Use contact numbers, not an assumed solder-side drawing. Pins 1, 2, 3 have NO PCB connection. Insulate DIN shell from metal enclosure; leave open."
- note removed: "Female DIN, 180 degrees. Use contact numbers, not an assumed solder-side drawing. Pins 1, 2, 3 have NO PCB connection. Metal shell bonded to enclosure mechanically."
