File: hardware/aaa/ardor-io/03_Expression.kicad_sch (KiCad schematic)
At the start: 21 parts, among them J301 EXPRESSION / 6.3mm TRS, J302 TO EXP PANEL / T,R,S, U301 ADS1115IDGS

Commit message: feat: finalize Ardor IO hardware rev2 production package
- Update schematics, PCB, BOM, and documentation
- Add assembly exports, review artifacts, and verification data
Parts:
- C301, C302, C303: value 100n / 16V -> 100n / 50V X7R; JLCPCB Part # (none) -> C14663; MPN (none) -> YAGEO CC0603KRX7R9BB104
- D301, D302: JLCPCB Part # (none) -> C19224; MPN Nexperia PESD5V0S1BA -> Nexperia PESD5V0S1BA,115
- D303, D304, D305, D306: JLCPCB Part # (none) -> C426769
- R301: JLCPCB Part # (none) -> C21190; MPN (none) -> UNI-ROYAL 0603WAF1001T5E
- R302, R304: JLCPCB Part # (none) -> C25804; MPN (none) -> UNI-ROYAL 0603WAF1002T5E
- R303: JLCPCB Part # (none) -> C22935; MPN (none) -> UNI-ROYAL 0603WAF1004T5E
- R305, R306: JLCPCB Part # (none) -> C23140; MPN (none) -> UNI-ROYAL 0603WAF330JT5E
- R307: JLCPCB Part # (none) -> C4190; MPN (none) -> UNI-ROYAL 0603WAF2201T5E
- U301: JLCPCB Part # (none) -> C37593
Other:
- note added: "TVS at jack entry; R302 then clamp pair at ADC. R301 limits insertion/short current to <=3.5 mA. Passive pedals only; no powered CV source. Calibrate endpoints; pot loading remains nonlinear."
- note removed: "TVS at jack entry; R302 then clamp pair at ADC. R301 limits insertion/short current to <=3.5 mA. Passive pedals only; no powered CV source. Calibrate endpoints to remove pot loading error."
