File: hardware/aaa/ardor-io/06_Headphones.kicad_sch (KiCad schematic)
At the start: 17 parts, among them J601 HEADPHONES / 3.5mm TRS, J602 TO HP PANEL / T,R,S, U601 TPA6132A2RTER

Commit message: feat: smd capacitors
Parts:
- C601, C602: value 2.2u / 63V film -> 2.2u / 16V film; footprint Capacitor_THT:C_Rect_L7.2mm_W7.2mm_P5.00mm_FKS2_FKP2_MKS2_MKP2 -> Ardor_Capacitor:C_Rubycon_MU_3225; MPN WIMA MKS2C042201K00KSSD -> Rubycon 16MU225KB23225

Commit message: feat: update Ardor IO PCB for hardware rev2
- Update schematics, routing, BOM, and design documentation
- Add SMD capacitor conversion and verification tooling
Parts:
- C601, C602: value 2.2u / 16V film -> 10u / 50V X7R; footprint Ardor_Capacitor:C_Rubycon_MU_3225 -> Capacitor_SMD:C_1206_3216Metric; JLCPCB Part # (none) -> C89632; MPN Rubycon 16MU225KB23225 -> Samsung CL31B106KBHNNNE

Commit message: feat: finalize Ardor IO hardware rev2 production package
- Update schematics, PCB, BOM, and documentation
- Add assembly exports, review artifacts, and verification data
Parts:
- C603, C605, C606, C607: value 2.2u / 10V X7R -> 2.2u / 25V X7R; JLCPCB Part # (none) -> C19110; MPN (none) -> Samsung CL21B225KAFNNNE
- C604: value 100n / 16V -> 100n / 50V X7R; JLCPCB Part # (none) -> C14663; MPN (none) -> YAGEO CC0603KRX7R9BB104
- D601, D602: JLCPCB Part # (none) -> C19224; MPN Nexperia PESD5V0S1BA -> Nexperia PESD5V0S1BA,115
- R601: JLCPCB Part # (none) -> C21190; MPN (none) -> UNI-ROYAL 0603WAF1001T5E
- R602: JLCPCB Part # (none) -> C25803; MPN (none) -> UNI-ROYAL 0603WAF1003T5E
- R603, R604: JLCPCB Part # (none) -> C22939; MPN (none) -> UNI-ROYAL 0603WAF220KT5E
- U601: JLCPCB Part # (none) -> C69901
