File: hardware/aaa/ardor-io/Ardor_IO.kicad_sch (KiCad schematic)
At the start: 12 parts, among them J101 PI 40-PIN HEADER, J102 CODEC AUX L / GND / R

Commit message: feat: finalize Ardor IO hardware rev2 production package
- Update schematics, PCB, BOM, and documentation
- Add assembly exports, review artifacts, and verification data
Parts:
- C101: JLCPCB Part # (none) -> C907991; MPN (none) -> Murata GRM21BZ71A226ME15L
- C102, C104: value 100n / 16V -> 100n / 50V X7R; JLCPCB Part # (none) -> C14663; MPN (none) -> YAGEO CC0603KRX7R9BB104
- C103: value 10u / 10V X7R -> 10u / 16V X7R; JLCPCB Part # (none) -> C95841; MPN (none) -> Samsung CL21B106KOQNNNE
- FB101: JLCPCB Part # (none) -> C41556732
- FB102: JLCPCB Part # (none) -> C19330
- R101: JLCPCB Part # (none) -> C17888; MPN (none) -> UNI-ROYAL 1206W4F0000T5E
Other:
- note added: "Audio jack sleeves bond GND to aluminium enclosure. Use one continuous PCB ground plane; place by function. R101 bonds TVS CHASSIS to GND; keep sleeve leads short. 5 V source: 4.75-5.25 V; reserve 150 mA beyond Pi/Codec. Pi provides 3.3 V. No second supply or USB back-feed."
- note removed: "Bond enclosure at connector entry. Short, wide copper. Use one continuous PCB ground plane; place by function. Do not route ESD or charge-pump return through ADC/audio. 5 V source: 4.75-5.25 V; reserve 150 mA beyond Pi/Codec. Pi provides 3.3 V. No second supply or USB back-feed."
