File: hardware/aaa/ardor-io-revc/Ardor_IO.kicad_pcb (KiCad board)
At the start: 2 copper layers, 68 x 46 mm, 81 parts, among them J101 PI 40-PIN HEADER, J102 CODEC AUX L / GND / R, J202 TO MIDI PANEL / 4,5, J302 TO EXP PANEL / T,R,S, J502 TO YOUR AMP CIRCUIT, J503 TO LINE PANEL / T,S, K501 G5V-1 DC5, Q501 AO3400A, U201 H11L1M, U301 ADS1115IDGS, U401 TLV9002IDR, U402 TLV9002IDR

Commit message: feat: changes to the layout
Parts:
- moved R501 10.7 mm to (100.1, 67.6), turned to 0 degrees
- moved TP402 8.06 mm to (103.2, 81.2)
- moved C402 7.65 mm to (62.5, 62.6)
- moved R405 7.24 mm to (94.2, 77.0), turned to 180 degrees
- moved TP101 6.09 mm to (90.5, 67.2)
- moved TP301 6.06 mm to (69.2, 87.9)
- moved C302 2.82 mm to (72.5, 87.8), turned to 0 degrees
- moved R406 2.75 mm to (88.2, 77.0), turned to 180 degrees
- moved D306 2.58 mm to (77.7, 90.0)
- moved C403 2.17 mm to (91.1, 77.9), turned to -90 degrees
- moved C401 2.16 mm to (62.5, 59.9)
- moved R402 1.93 mm to (83.2, 71.5), turned to -90 degrees
- moved R307 1.91 mm to (76.5, 87.8), turned to 180 degrees
- moved R201 1.47 mm to (64.2, 67.3), turned to 0 degrees
- moved TP201 1.27 mm to (79.2, 76.0)
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Routing:
- net +5V_A: track 61.3 -> 44.0 mm
- net MONO_BUF: track 50.1 -> 37.5 mm, vias 4 -> 2
- net AUX_R: track 11.3 -> 3.17 mm
- net /05 / Line and amp feed/LINE_AC: track 17.9 -> 9.85 mm
- net CHASSIS: track 126.8 -> 121.2 mm, vias 4 -> 2
- net EXP_ADC: track 23.5 -> 19.8 mm
- net MIDI_4: track 15.2 -> 11.7 mm
- net +3V3_ADC: track 62.5 -> 59.4 mm
- net VREF_DIV: track 9.43 -> 6.84 mm
- net MIDI_A: track 14.2 -> 12.2 mm
- net /04 / Audio distribution/BUF_R: track 7.27 -> 5.51 mm
- net /04 / Audio distribution/BIAS_L: track 17.9 -> 19.3 mm
- net MIDI_4_F: track 4.08 -> 2.64 mm
- net EXP_RING: track 18.8 -> 20.2 mm
- net GND: track 4.65 -> 3.44 mm
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