File: hardware/aaa/ardor-modules/expression/Ardor_Expression.kicad_pcb (KiCad board)
At the start: 2 copper layers, 44 x 34 mm, 31 parts, among them J101 +3V3 / GND / SDA / SCL, J302 EXP_TIP / EXP_RING / GND, U301 ADS1115IDGSR

Commit message: feat: clarify module pin labels and add STE assembly guides
Parts:
- J101: value +3V3 / GND / SDA / SCL -> 3V3 POWER INPUT + I2C TO HOST
- J302: value EXP_TIP / EXP_RING / GND -> PASSIVE PEDAL INPUT / EXCITATION OUTPUT
- JP301: value TIP/RING / TWO SHUNTS -> JUMPER ONLY: PEDAL POLARITY
- JP302: value GND / ADDR / +3V3_A -> JUMPER ONLY: ADC ADDRESS
- JP303: value SDA_PULL / SDA -> JUMPER ONLY: SDA PULLUP
- JP304: value SCL_PULL / SCL -> JUMPER ONLY: SCL PULLUP
Other:
- board text added: "1"
- board text added: "2"
- board text added: "3"
- board text added: "4"
- board text added: "5"
- board text added: "6"
- board text added: "I/O=BOTH"
- board text added: "IN=INTO"
- board text added: "J101 PWR IN / I2C 1 3V3 IN 2 GND 0V 3 DATA I/O 4 CLOCK IN"
- board text added: "J302 PASSIVE PEDAL 1 TIP I/O 2 RING I/O 3 GND 0V"
- board text added: "JP301 PEDAL JUMPER 1 TIP 2 RING 3 PEDAL IN 4 EXC OUT 5 RING 6 TIP"
- board text added: "JP302 ADDR JUMPER 1 LOW GND 2 SELECT 3 HIGH 3V3"
- board text added: "JP303 DATA PULLUP 1 PULLUP 2 DATA I/O"
- board text added: "JP304 CLOCK PULLUP 1 PULLUP 2 CLOCK IN"
- board text added: "JP=SHUNTS"
- board text added: "OUT=FROM"
- board text added: "U301.2 NC NO WIRE"
- board text removed: "3V3"
- board text removed: "GND"
- board text removed: "J302: 1=T 2=R 3=G"
- board text removed: "SCL"
- board text removed: "SDA"
