File: hardware/aaa/ardor-modules/expression/Ardor_Expression.kicad_sch (KiCad schematic)
At the start: 29 parts, among them J101 +3V3 / GND / SDA / SCL, J302 EXP_TIP / EXP_RING / GND, U301 ADS1115IDGSR

Commit message: feat: clarify module pin labels and add STE assembly guides
Parts:
- J101: value +3V3 / GND / SDA / SCL -> 3V3 POWER INPUT + I2C TO HOST
- J302: value EXP_TIP / EXP_RING / GND -> PASSIVE PEDAL INPUT / EXCITATION OUTPUT
- JP301: value TIP/RING / TWO SHUNTS -> JUMPER ONLY: PEDAL POLARITY
- JP302: value GND / ADDR / +3V3_A -> JUMPER ONLY: ADC ADDRESS
- JP303: value SDA_PULL / SDA -> JUMPER ONLY: SDA PULLUP
- JP304: value SCL_PULL / SCL -> JUMPER ONLY: SCL PULLUP
Other:
- note added: "1: 3V3 IN 2: GND 0V"
- note added: "1: LOW GND 2: SELECT"
- note added: "1: PULLUP 2: CLOCK IN"
- note added: "1: PULLUP 2: DATA I/O"
- note added: "1: TIP 2: RING"
- note added: "1: TIP I/O 2: RING I/O"
- note added: "3: DATA I/O 4: CLOCK IN"
- note added: "3: GND 0V"
- note added: "3: HIGH 3V3"
- note added: "3: PEDAL IN 4: EXC OUT"
- note added: "5: RING 6: TIP"
- note added: "J101 / PWR IN / I2C"
- note added: "J302 / PASSIVE PEDAL"
- note added: "JP301 / PEDAL JUMPER"
- note added: "JP302 / ADDR JUMPER"
- note added: "JP303 / DATA PULLUP"
- note added: "JP304 / CLOCK PULLUP"
- note added: "M1 | INDEPENDENT MODULE | SEE PIN GUIDE AT RIGHT"
- note added: "PIN GUIDE: IN = into this board / OUT = out / I/O = both / GND = 0 V"
- note added: "U301.2: UNUSED ALERT - LEAVE OPEN"
- note removed: "REV M1 | EXTERNAL HOST + REGULATED POWER | NO OTHER MODULE REQUIRED"
