File: hardware/aaa/ardor-modules/headphones/Ardor_Headphones.kicad_pcb (KiCad board)
At the start: 2 copper layers, 36 x 30 mm, 23 parts, among them J101 +5V / GND / HP_ENABLE, J102 AUDIO_L / GND / AUDIO_R, J602 HP_L / HP_R / GND, U601 TPA6132A2RTER

Commit message: feat: clarify module pin labels and add STE assembly guides
Parts:
- J101: value +5V / GND / HP_ENABLE -> 5V POWER + ENABLE INPUT
- J102: value AUDIO_L / GND / AUDIO_R -> STEREO AUDIO INPUT FROM SOURCE
- J602: value HP_L / HP_R / GND -> STEREO HEADPHONE AUDIO OUTPUT
Other:
- board text added: "1"
- board text added: "2"
- board text added: "3"
- board text added: "IN=INTO"
- board text added: "J101 PWR + ENABLE IN 1 5V IN 2 GND 0V 3 ENABLE IN"
- board text added: "J102 AUDIO IN 1 LEFT IN 2 GND 0V 3 RIGHT IN"
- board text added: "J602 HEADPHONE OUT 1 LEFT OUT 2 RIGHT OUT 3 GND 0V"
- board text added: "OUT=FROM"
- board text removed: "5V"
- board text removed: "EN"
- board text removed: "GND"
- board text removed: "L"
- board text removed: "R"
