File: hardware/aaa/ardor-modules/line-out/Ardor_Line_Out.kicad_pcb (KiCad board)
At the start: 2 copper layers, 46 x 34 mm, 29 parts, among them J101 +5V / GND / LINE_ENABLE, J102 AUDIO_IN / GND, J502 AMP_FEED / GND, J503 LINE_JACK / GND, K501 Omron G5V-1 DC5, Q501 AO3400A, U501 TLV9002IDR

Commit message: feat: clarify module pin labels and add STE assembly guides
Parts:
- J101: value +5V / GND / LINE_ENABLE -> 5V POWER + ENABLE INPUT
- J102: value AUDIO_IN / GND -> MONO AUDIO INPUT FROM SOURCE
- J502: value AMP_FEED / GND -> AUDIO OUTPUT TO AMP INPUT
- J503: value LINE_JACK / GND -> LINE AUDIO OUTPUT TO TS SOCKET
Other:
- board text added: "1"
- board text added: "2"
- board text added: "3"
- board text added: "IN=INTO"
- board text added: "J101 PWR + ENABLE IN 1 5V IN 2 GND 0V 3 ENABLE IN"
- board text added: "J102 AUDIO IN 1 AUDIO IN 2 GND 0V"
- board text added: "J502 AMP AUDIO OUT 1 AUDIO OUT 2 GND 0V"
- board text added: "J503 LINE OUT 1 LINE OUT 2 GND 0V"
- board text added: "OUT=FROM"
- board text removed: "5V"
- board text removed: "AMP"
- board text removed: "EN"
- board text removed: "GND"
- board text removed: "IN"
- board text removed: "OUT"
