File: hardware/aaa/ardor-modules/line-out/Ardor_Line_Out.kicad_sch (KiCad schematic)
At the start: 27 parts, among them J101 +5V / GND / LINE_ENABLE, J102 AUDIO_IN / GND, J502 AMP_FEED / GND, J503 LINE_JACK / GND, K501 Omron G5V-1 DC5, Q501 AO3400A, U501 TLV9002IDR

Commit message: feat: clarify module pin labels and add STE assembly guides
Parts:
- J101: value +5V / GND / LINE_ENABLE -> 5V POWER + ENABLE INPUT
- J102: value AUDIO_IN / GND -> MONO AUDIO INPUT FROM SOURCE
- J502: value AMP_FEED / GND -> AUDIO OUTPUT TO AMP INPUT
- J503: value LINE_JACK / GND -> LINE AUDIO OUTPUT TO TS SOCKET
Other:
- note added: "1: 5V IN 2: GND 0V"
- note added: "1: AUDIO IN 2: GND 0V"
- note added: "1: AUDIO OUT 2: GND 0V"
- note added: "1: LINE OUT 2: GND 0V"
- note added: "3: ENABLE IN"
- note added: "J101 / PWR + ENABLE IN"
- note added: "J102 / AUDIO IN"
- note added: "J502 / AMP AUDIO OUT"
- note added: "J503 / LINE OUT"
- note added: "M1 | INDEPENDENT MODULE | SEE PIN GUIDE AT RIGHT"
- note added: "PIN GUIDE: IN = into this board / OUT = out / I/O = both / GND = 0 V"
- note removed: "REV M1 | EXTERNAL HOST + REGULATED POWER | NO OTHER MODULE REQUIRED"
