File: hardware/aaa/ardor-modules/midi-in/Ardor_MIDI.kicad_pcb (KiCad board)
At the start: 2 copper layers, 34 x 28 mm, 20 parts, among them J101 +5V / +3V3 / GND / MIDI_RX, J202 MIDI_4 / MIDI_5, J203 CHASSIS / GND, U201 onsemi H11L1M

Commit message: feat: clarify module pin labels and add STE assembly guides
Parts:
- J101: value +5V / +3V3 / GND / MIDI_RX -> POWER INPUT + UART OUTPUT TO HOST
- J202: value MIDI_4 / MIDI_5 -> MIDI INPUT FROM DIN SOCKET
- J203: value CHASSIS / GND -> METAL CASE BOND + GROUND
Other:
- board text added: "1"
- board text added: "2"
- board text added: "3"
- board text added: "IN=INTO"
- board text added: "J101 PWR IN / UART OUT 1 5V IN 2 3V3 IN 3 GND 0V 4 UART OUT"
- board text added: "J202 MIDI IN 1 DIN4 IN 2 DIN5 IN"
- board text added: "J203 CASE BOND 1 CASE 2 GND 0V"
- board text added: "OUT=FROM"
- board text added: "U201.3 NC NO WIRE"
- board text removed: "3V3"
- board text removed: "5"
- board text removed: "5V"
- board text removed: "CHS"
- board text removed: "GND"
- board text removed: "RX"
