File: hardware/aaa/ardor-modules/midi-in/Ardor_MIDI.kicad_sch (KiCad schematic)
At the start: 18 parts, among them J101 +5V / +3V3 / GND / MIDI_RX, J202 MIDI_4 / MIDI_5, J203 CHASSIS / GND, U201 onsemi H11L1M

Commit message: feat: clarify module pin labels and add STE assembly guides
Parts:
- J101: value +5V / +3V3 / GND / MIDI_RX -> POWER INPUT + UART OUTPUT TO HOST
- J202: value MIDI_4 / MIDI_5 -> MIDI INPUT FROM DIN SOCKET
- J203: value CHASSIS / GND -> METAL CASE BOND + GROUND
Other:
- note added: "1: 5V IN 2: 3V3 IN"
- note added: "1: CASE 2: GND 0V"
- note added: "1: DIN4 IN 2: DIN5 IN"
- note added: "3: GND 0V 4: UART OUT"
- note added: "J101 / PWR IN / UART OUT"
- note added: "J202 / MIDI IN"
- note added: "J203 / CASE BOND"
- note added: "M1 | INDEPENDENT MODULE | SEE PIN GUIDE AT RIGHT"
- note added: "PIN GUIDE: IN = into this board / OUT = out / I/O = both / GND = 0 V"
- note added: "U201.3: NC - LEAVE OPEN"
- note removed: "REV M1 | EXTERNAL HOST + REGULATED POWER | NO OTHER MODULE REQUIRED"
