File: hardware/aaa/ardor-modules/mixer/Ardor_Mixer.kicad_pcb (KiCad board)
At the start: 2 copper layers, 40 x 30 mm, 30 parts, among them J101 +5V / GND, J102 AUDIO_L / GND / AUDIO_R, J103 OUT_L / GND / OUT_R / OUT_MONO, U401 TLV9002IDR, U402 TLV9002IDR

Commit message: feat: clarify module pin labels and add STE assembly guides
Parts:
- J101: value +5V / GND -> 5V POWER INPUT
- J102: value AUDIO_L / GND / AUDIO_R -> STEREO AUDIO INPUT FROM SOURCE
- J103: value OUT_L / GND / OUT_R / OUT_MONO -> BUFFERED STEREO + MONO AUDIO OUTPUT
Other:
- board text added: "1"
- board text added: "2"
- board text added: "3"
- board text added: "4"
- board text added: "IN=INTO"
- board text added: "J101 POWER IN 1 5V IN 2 GND 0V"
- board text added: "J102 AUDIO IN 1 LEFT IN 2 GND 0V 3 RIGHT IN"
- board text added: "J103 AUDIO OUT 1 LEFT OUT 2 GND 0V 3 RIGHT OUT 4 MONO OUT"
- board text added: "OUT=FROM"
- board text removed: "5V"
- board text removed: "GND"
- board text removed: "L"
- board text removed: "MONO"
- board text removed: "R"
