File: hardware/aaa/ardor-modules/mixer/Ardor_Mixer.kicad_sch (KiCad schematic)
At the start: 28 parts, among them J101 +5V / GND, J102 AUDIO_L / GND / AUDIO_R, J103 OUT_L / GND / OUT_R / OUT_MONO, U401 TLV9002IDR, U402 TLV9002IDR

Commit message: feat: clarify module pin labels and add STE assembly guides
Parts:
- J101: value +5V / GND -> 5V POWER INPUT
- J102: value AUDIO_L / GND / AUDIO_R -> STEREO AUDIO INPUT FROM SOURCE
- J103: value OUT_L / GND / OUT_R / OUT_MONO -> BUFFERED STEREO + MONO AUDIO OUTPUT
Other:
- note added: "1: 5V IN 2: GND 0V"
- note added: "1: LEFT IN 2: GND 0V"
- note added: "1: LEFT OUT 2: GND 0V"
- note added: "3: RIGHT IN"
- note added: "3: RIGHT OUT 4: MONO OUT"
- note added: "J101 / POWER IN"
- note added: "J102 / AUDIO IN"
- note added: "J103 / AUDIO OUT"
- note added: "M1 | INDEPENDENT MODULE | SEE PIN GUIDE AT RIGHT"
- note added: "PIN GUIDE: IN = into this board / OUT = out / I/O = both / GND = 0 V"
- note removed: "REV M1 | EXTERNAL HOST + REGULATED POWER | NO OTHER MODULE REQUIRED"
