File: hardware/aaa/ardor-modules-tht/mixer/Ardor_Mixer_THT.kicad_sch (KiCad schematic)
At the start: 28 parts, among them J101 5V POWER INPUT, J102 STEREO AUDIO INPUT FROM SOURCE, J103 BUFFERED STEREO + MONO AUDIO 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, U401 MCP6022-I/P, U402 MCP6022-I/P

Commit message: feat(hardware): compact layouts and adopt Hestore module packages
Parts:
- C401, C402, C407, C408, C409: value 10u / 25V BIPOLAR -> 10u / 50V BIPOLAR; footprint Ardor_THT:CP_Bipolar_D6.3mm_P2.50mm -> Ardor_THT:CP_Bipolar_Nichicon_D8.0mm_P3.50mm; MPN Nichicon UES1E100MDM -> Nichicon UES1H100MPM (HESTORE 100.524.69)
